File: mp3_fa2026.kicad_pcb (KiCad board)
At the start: 2 copper layers, 29.6 x 51.4 mm, 41 parts, among them J1 USB4105-GF-A, J2 LEFT, J3 RIGHT, J4 DEBUG, U1 RP2354A, U2 MCP1702T-3302E_CB, X1 IQXO-791_12MHz

Commit message: Work on mp3
Routing:
- net GND: track 67.9 -> 70.5 mm, vias 39 -> 51
Changed lines of the file:
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@@
 	)
 	(segment
+		(start 143.129 117.221)
+		(end 143.1536 117.221)
+		(width 0.1524)
+		(layer "F.Cu")
+		(net "GND")
+	)
+	(segment
 		(start 154.94 82.897)
 		(end 152.62 82.897)
@@
 	)
 	(segment
+		(start 138.815 107.53)
+		(end 138.815 107.438)
+		(width 0.1524)
+		(layer "F.Cu")
+		(net "GND")
+	)
+	(segment
 		(start 141.215 102.13)
 		(end 141.491 101.854)
@@
 	)
 	(segment
+		(start 138.815 107.53)
+		(end 138.815 107.573)
+		(width 0.1524)
+		(layer "F.Cu")
+		(net "GND")
+	)
+	(segment
 		(start 135.001 100.571)
 		(end 135.001 100.33)
@@
 	)
 	(segment
+		(start 139.915 107.53)
+		(end 139.954 107.569)
+		(width 0.1524)
+		(layer "F.Cu")
+		(net "GND")
+	)
+	(segment
 		(start 136.79 83.174)
 		(end 135.636 84.328)
@@
 	)
 	(segment
+		(start 140.843 117.094)
+		(end 140.843 117.221)
+		(width 0.1524)
+		(layer "F.Cu")
+		(net "GND")
+	)
+	(segment
+		(start 143.1536 119.3554)
+		(end 143.129 119.38)
+		(width 0.1524)
+		(layer "F.Cu")
+		(net "GND")
+	)
+	(segment
 		(start 148.082 122.301)
 		(end 148.365 122.301)
@@
 	)
 	(segment
-		(start 140.882 107.53)
-		(end 138.815 107.53)
-		(width 0.1524)
-		(layer "F.Cu")
-		(net "GND")
-	)
-	(segment
 		(start 131.032211 105.243553)
 		(end 131.813 106.024342)
@@
 	)
 	(segment
+		(start 138.815 106.303)
+		(end 138.811 106.299)
+		(width 0.1524)
+		(layer "F.Cu")
+		(net "GND")
+	)
+	(segment
+		(start 138.815 108.581)
+		(end 138.811 108.585)
+		(width 0.1524)
+		(layer "F.Cu")
+		(net "GND")
+	)
+	(segment
 		(start 143.764 94.488)
 		(end 143.764 94.107)
@@
 	)
 	(segment
+		(start 140.716 119.507)
+		(end 140.716 117.221)
+		(width 0.1524)
+		(layer "F.Cu")
+		(net "GND")
+	)
+	(segment
 		(start 154.178 121.759)
 		(end 154.94 120.997)
@@
 	)
 	(segment
+		(start 138.815 107.53)
+		(end 138.723 107.53)
+		(width 0.1524)
+		(layer "F.Cu")
+		(net "GND")
+	)
+	(segment
 		(start 146.928 83.174)
 		(end 147.32 83.566)
@@
 	)
 	(segment
-		(start 141.139185 107.399028)
-		(end 141.012972 107.399028)
+		(start 134.848 113.962)
+		(end 135.186 114.3)
 		(width 0.1524)
 		(layer "F.Cu")
@@
 	)
 	(segment
-		(start 134.848 113.962)
-		(end 135.186 114.3)
+		(start 133.35 102.082)
+		(end 133.35 100.965)
 		(width 0.1524)
 		(layer "F.Cu")
@@
 	)
 	(segment
-		(start 133.35 102.082)
-		(end 133.35 100.965)
+		(start 137.58 107.53)
+		(end 137.541 107.569)
 		(width 0.1524)
 		(layer "F.Cu")
@@
 	)
 	(segment
-		(start 134.239 118.123)
-		(end 134.252 118.123)
+		(start 143.1536 117.221)
+		(end 143.1536 119.3554)
 		(width 0.1524)
 		(layer "F.Cu")
@@
 	)
 	(segment
-		(start 149.86 90.205)
-		(end 151.292 90.205)
+		(start 134.239 118.123)
+		(end 134.252 118.123)
 		(width 0.1524)
 		(layer "F.Cu")
@@
 	)
 	(segment
-		(start 141.012972 107.399028)
-		(end 140.882 107.53)
+		(start 149.86 90.205)
+		(end 151.292 90.205)
 		(width 0.1524)
 		(layer "F.Cu")
@@
 	)
 	(via
+		(at 137.541 107.569)
+		(size 0.6096)
+		(drill 0.3048)
+		(layers "F.Cu" "B.Cu")
+		(net "GND")
+	)
+	(via
 		(at 137.922 118.364)
 		(size 0.6096)
@@
 	)
 	(via
+		(at 143.129 119.38)
+		(size 0.6096)
+		(drill 0.3048)
+		(layers "F.Cu" "B.Cu")
+		(free yes)
+		(net "GND")
+	)
+	(via
 		(at 154.178 122.174)
 		(size 0.6096)
@@
 	)
 	(via
-		(at 141.139185 107.399028)
+		(at 137.541 108.712)
+		(size 0.6096)
+		(drill 0.3048)
+		(layers "F.Cu" "B.Cu")
+		(net "GND")
+	)
+	(via
+		(at 137.541 106.299)
 		(size 0.6096)
 		(drill 0.3048)
@@
 	)
 	(via
+		(at 138.815 107.53)
+		(size 0.6096)
+		(drill 0.3048)
+		(layers "F.Cu" "B.Cu")
+		(net "GND")
+	)
+	(via
 		(at 151.257 95.377)
 		(size 0.6096)
@@
 	)
 	(via
+		(at 139.954 107.569)
+		(size 0.6096)
+		(drill 0.3048)
+		(layers "F.Cu" "B.Cu")
+		(net "GND")
+	)
+	(via
 		(at 155.829 107.188)
 		(size 0.6096)
@@
 	)
 	(via
+		(at 140.716 119.507)
+		(size 0.6096)
+		(drill 0.3048)
+		(layers "F.Cu" "B.Cu")
+		(net "GND")
+	)
+	(via
 		(at 135.636 78.994)
 		(size 0.6096)
@@
 	)
 	(via
+		(at 138.811 106.299)
+		(size 0.6096)
+		(drill 0.3048)
+		(layers "F.Cu" "B.Cu")
+		(net "GND")
+	)
+	(via
 		(at 147.32 107.061)
 		(size 0.6096)
@@
 	)
 	(via
+		(at 140.716 117.221)
+		(size 0.6096)
+		(drill 0.3048)
+		(layers "F.Cu" "B.Cu")
+		(net "GND")
+	)
+	(via
 		(at 135.186 114.3)
 		(size 0.6096)
@@
 	)
 	(via
+		(at 143.1536 117.221)
+		(size 0.6096)
+		(drill 0.3048)
+		(layers "F.Cu" "B.Cu")
+		(free yes)
+		(net "GND")
+	)
+	(via
+		(at 139.954 108.712)
+		(size 0.6096)
+		(drill 0.3048)
+		(layers "F.Cu" "B.Cu")
+		(net "GND")
+	)
+	(via
+		(at 138.811 108.712)
+		(size 0.6096)
+		(drill 0.3048)
+		(layers "F.Cu" "B.Cu")
+		(net "GND")
+	)
+	(via
 		(at 147.066 78.994)
 		(size 0.6096)
@@
 		(net "GND")
 	)
+	(via
+		(at 139.954 106.299)
+		(size 0.6096)
+		(drill 0.3048)
+		(layers "F.Cu" "B.Cu")
+		(net "GND")
+	)
 	(segment
 		(start 149.128 93.726)
@@
 	)
 	(segment
-		(start 139.615 112.258452)
-		(end 140.1572 112.800652)
+		(start 140.081 115.680006)
+		(end 140.081 119.133658)
 		(width 0.1524)
 		(layer "F.Cu")
@@
 	)
 	(segment
-		(start 139.615 111.03)
-		(end 139.615 112.258452)
+		(start 140.081 119.133658)
+		(end 140.0556 119.159058)
+		(width 0.1524)
+		(layer "F.Cu")
+		(net "/SWDIO")
+	)
+	(segment
+		(start 140.0556 119.159058)
+		(end 140.0556 122.0216)
+		(width 0.1524)
+		(layer "F.Cu")
+		(net "/SWDIO")
+	)
+	(segment
+		(start 139.615 112.258452)
+		(end 140.1572 112.800652)
 		(width 0.1524)
 		(layer "F.Cu")
@@
 	(segment
 		(start 140.1572 115.603806)
-		(end 140.0302 115.730806)
+		(end 140.081 115.680006)
 		(width 0.1524)
 		(layer "F.Cu")
@@
 	)
 	(segment
-		(start 140.0302 115.730806)
-		(end 140.0302 121.9962)
+		(start 139.615 111.03)
+		(end 139.615 112.258452)
 		(width 0.1524)
 		(layer "F.Cu")
@@
 	)
 	(segment
-		(start 140.0302 121.9962)
+		(start 140.0556 122.0216)
 		(end 144.018 125.984)
 		(width 0.1524)
